File: KiCad10_KiBot_Template.kicad_pcb (KiCad board)
At the start: 4 copper layers, 0 parts

Commit message: Starter board, JLCPCB order files, PR checks, outputs branch, --init
- Starter board: 40x30 mm outline, H1-H4 mounting holes, TP1 on GND
  (ERC/DRC/parity clean), real dimensions, so every status works from the
  first run. KDT example dimensions for another board removed.
- Impedance tables from the JLCPCB calculator, stored in the stackup
  profiles and written by --stackup (JLC04161H-7628 / JLC06161H-3313).
- JLCPCB order files (KiBot JLCPCB template): Gerbers ZIP, BoM with LCSC
  part numbers, pick and place with rotation corrections. LCSC column in
  the regular BoMs.
- CI: pull request checks (pr_variant, ERC/DRC) with a summary comment,
  job summary on every run, outputs published to kibot-outputs/<branch>
  (ci_outputs: branch | commit | none) instead of growing the history.
- ./run_kibot.sh --init sets the metadata and renames the project files;
  GIT_URL: auto uses the git remote. DRAFT README generated after the text
  variables update.
- Generated outputs committed by the first CI runs removed from the template.

Co-Authored-By: Claude Opus 5.5 (1M context) <noreply@anthropic.com>
Parts:
- added H1: M3, MountingHole:MountingHole_3.2mm_M3, F.Cu at (133.5, 73.5)
- added H2: M3, MountingHole:MountingHole_3.2mm_M3, F.Cu at (166.5, 73.5)
- added H3: M3, MountingHole:MountingHole_3.2mm_M3, F.Cu at (133.5, 96.5)
- added H4: M3, MountingHole:MountingHole_3.2mm_M3, F.Cu at (166.5, 96.5)
- added TP1: GND, TestPoint:TestPoint_THTPad_D1.5mm_Drill0.7mm, F.Cu at (150.0, 95.0)
Other:
- board outline added: 40 x 30 mm
- board text removed: "30°"
- board text removed: "3× 120°"
- board text removed: "X"
- board text removed: "Y"
